File: Hardware/SparkFun_Ambient_Light_Sensor_VEML6030.brd (EAGLE design)
At the start: 25.4 x 25.4 mm, 50 parts, among them U1 VEML6030

Commit message: Changed "Default" silk with "Open"
Parts:
- U$21: device Address text:DEFAULT#2 -> OPEN:OPEN#0
- moved U$21 0.21 mm to (16.0, 14.5)
Changed lines of the file:
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@@
 <layer number="115" name="ReferenceISLANDS" color="7" fill="1" visible="no" active="no"/>
 <layer number="116" name="Patch_BOT" color="9" fill="4" visible="no" active="no"/>
-<layer number="117" name="PM_Ref" color="26" fill="1" visible="yes" active="yes"/>
+<layer number="117" name="PM_Ref" color="26" fill="1" visible="no" active="yes"/>
 <layer number="118" name="Rect_Pads" color="7" fill="1" visible="no" active="no"/>
-<layer number="119" name="PF_Ref" color="31" fill="1" visible="yes" active="yes"/>
-<layer number="120" name="WFL_Ref" color="25" fill="1" visible="yes" active="yes"/>
+<layer number="119" name="PF_Ref" color="31" fill="1" visible="no" active="yes"/>
+<layer number="120" name="WFL_Ref" color="25" fill="1" visible="no" active="yes"/>
 <layer number="121" name="_tsilk" color="7" fill="1" visible="no" active="no"/>
 <layer number="122" name="_bsilk" color="7" fill="1" visible="no" active="no"/>
@@
 <element name="U$22" library="Address text" package="0X481" value="" x="9.8044" y="14.2748" smashed="yes" rot="MR0"/>
 <element name="U$24" library="Address text" package="0X103" value="" x="9.6012" y="12.7254" smashed="yes" rot="MR0"/>
-<element name="U$21" library="Address text" package="DEFAULT#2" value="" x="16.0528" y="14.2748" smashed="yes" rot="MR0"/>
 <element name="U$25" library="ADR" package="ADR0" value="" x="16.002" y="16.002" smashed="yes" rot="MR0"/>
 <element name="U$26" library="ADR" package="JUMPER1" value="" x="11.7856" y="16.002" smashed="yes" rot="MR0"/>
 <element name="U$20" library="ADR" package="CLOSED#2" value="" x="16.0528" y="12.7508" smashed="yes" rot="MR0"/>
+<element name="U$21" library="OPEN" package="OPEN#0" value="" x="16.002" y="14.478" smashed="yes" rot="MR0"/>
 </elements>
 <signals>

Commit message: Centers SparkFun logo on the underside
Parts:
- moved LOGO1 1.02 mm to (12.4, 20.3)
- moved LOGO2 0.57 mm to (23.1, 18.5)
Changed lines of the file:
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@@
 <attribute name="VALUE" x="9.71566875" y="14.13" size="1" layer="27" rot="R270"/>
 </element>
-<element name="LOGO1" library="SparkFun-Aesthetics" package="SFE_LOGO_NAME_FLAME_.1" value="SFE_LOGO_NAME_FLAME.1_INCH" x="13.462" y="20.32" smashed="yes" rot="MR0"/>
+<element name="LOGO1" library="SparkFun-Aesthetics" package="SFE_LOGO_NAME_FLAME_.1" value="SFE_LOGO_NAME_FLAME.1_INCH" x="12.446" y="20.32" smashed="yes" rot="MR0"/>
 <element name="U$1" library="SparkFun-Aesthetics" package="QWIIC_5MM" value="QWIIC_LOGO_5MM" x="2.794" y="8.128" smashed="yes"/>
-<element name="LOGO2" library="SparkFun-Aesthetics" package="OSHW-LOGO-S" value="OSHW-LOGOS" x="22.86" y="19.05" smashed="yes" rot="MR0"/>
+<element name="LOGO2" library="SparkFun-Aesthetics" package="OSHW-LOGO-S" value="OSHW-LOGOS" x="23.114" y="18.542" smashed="yes" rot="MR0"/>
 <element name="R4" library="SparkFun-Resistors" package="0603" value="1k" x="2.5908" y="17.018" smashed="yes">
 <attribute name="NAME" x="2.5908" y="17.78" size="0.6096" layer="25" font="vector" ratio="20" align="bottom-center"/>
